File: small_compliant_drive/small_compliant_drive.kicad_sch (KiCad schematic)
At the start: 24 parts, among them Q1 EPC2014C, Q2 EPC2014C, Q3 EPC2014C, Q4 EPC2014C, Q5 EPC2014C, Q6 EPC2014C, U1 INA181, U2 INA181, U3 INA181, U4 TL431DBZ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

Commit message: v1 prototype done and bought
Parts:
- removed BT1: Battery_Cell, symbol Device:Battery_Cell
- removed R1, R2, R3: 1m, symbol Device:R_Shunt_US
- added C3, C4, C5: 0.1u, Capacitor_SMD:C_0603_1608Metric, symbol Device:C
- added J1, J3: Conn_01x03_Pin, Connector_PinSocket_2.54mm:PinSocket_1x03_P2.54mm_Vertical, symbol Connector:Conn_01x03_Pin
- added J2: Conn_01x06_Pin, Connector_PinHeader_2.54mm:PinHeader_1x06_P2.54mm_Vertical, symbol Connector:Conn_01x06_Pin
- added J4: Conn_01x02_Pin, Connector_AMASS:AMASS_XT30U-M_1x02_P5.0mm_Vertical, symbol Connector:Conn_01x02_Pin
- added J5: Conn_01x02_Pin, Connector_PinHeader_2.54mm:PinHeader_1x02_P2.54mm_Vertical, symbol Connector:Conn_01x02_Pin
- added R1, R2, R3: 1m, Resistor_SMD:R_2512_6332Metric, symbol Device:R_US
- added TP10: Vref, TestPoint:TestPoint_Pad_D2.0mm, symbol Connector:TestPoint
- added TP7: Via, TestPoint:TestPoint_Pad_D2.0mm, symbol Connector:TestPoint
- added TP8: Vib, TestPoint:TestPoint_Pad_D2.0mm, symbol Connector:TestPoint
- added TP9: Vic, TestPoint:TestPoint_Pad_D2.0mm, symbol Connector:TestPoint
- C1, C2: footprint (none) -> Capacitor_SMD:C_0603_1608Metric
- H1, H2, H3: footprint (none) -> MountingHole:MountingHole_3mm_Pad
- R4: footprint (none) -> Resistor_SMD:R_0603_1608Metric
- TP1, TP2, TP3: footprint (none) -> TestPoint:TestPoint_Pad_D2.0mm
Connections:
- net 3.3V: now also C3.1, C4.1, C5.1
- net Common: now also U5.7 (EP), C3.2, C4.2, C5.2, J4.2 (Pin_2), J5.1 (Pin_1), J5.2 (Pin_2)
- net Ia: now also J1.1 (Pin_1), TP7.1
- net Ib: now also J1.2 (Pin_2), TP8.1
- net Ic: now also J1.3 (Pin_3), TP9.1
- net PHASE_A_HIGH: now also J2.1 (Pin_1)
- net PHASE_A_LOW: now also J2.2 (Pin_2)
- net PHASE_B_HIGH: now also J2.3 (Pin_3)
- net PHASE_B_LOW: now also J2.4 (Pin_4)
- net PHASE_C_HIGH: now also J2.5 (Pin_5)
- net PHASE_C_LOW: now also J2.6 (Pin_6)
- net Vbat: now also J4.1 (Pin_1)
- net Vref: now also TP10.1
- net VsensA: now reaches H1.1
- net VsensA: now also U1.4 (-), J3.1 (Pin_1), R1.2
- net VsensC: now reaches H3.1
- net VsensC: now also U3.4 (-), J3.3 (Pin_3), R3.2
- net at Q5.2 (Sub), Q5.4 (S1), Q6.3 (D1)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: now also U3.3 (+), R3.1
- net at U1.3 (+): now also Q1.2 (Sub), Q1.4 (S1), Q2.3 (D1), Q2.5 (D2), R1.1
- net at Q3.2 (Sub), Q3.4 (S1), Q4.3 (D1)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: now also U2.3 (+), R2.1
- net VsensB: now reaches U2.4 (-)
- net VsensB: now also H2.1, J3.2 (Pin_2), R2.2
- no-connect marks 1 -> 0
Other:
- note added: "1.24V"
- note added: "This is the reference voltage for the current sensing. Voltages on the output lower than this one will be negative currents and vice versa."
